Commit message: fixed package name issue

File: urdf/mr_robot.xacro (robot description, xacro)
@@ -1,7 +1,7 @@
 <?xml version="1.0" ?>
 <robot name="mr_robot" xmlns:xacro="http://www.ros.org/wiki/xacro">
-<xacro:include filename="$(find linef)/urdf/materials.xacro" />
-<xacro:include filename="$(find linef)/urdf/mr_robot.trans" />
-<xacro:include filename="$(find linef)/urdf/mr_robot.gazebo" />
+<xacro:include filename="$(find line_follower_omnidrive)/urdf/materials.xacro" />
+<xacro:include filename="$(find line_follower_omnidrive)/urdf/mr_robot.trans" />
+<xacro:include filename="$(find line_follower_omnidrive)/urdf/mr_robot.gazebo" />
 <link name="base_link">
   <inertial>
@@ -13,5 +13,5 @@
     <origin xyz="0 0 0" rpy="0 0 0"/>
     <geometry>
-      <mesh filename="package://linef/models/robot/base_link.stl" scale="0.001 0.001 0.001"/>
+      <mesh filename="package://line_follower_omnidrive/models/robot/base_link.stl" scale="0.001 0.001 0.001"/>
     </geometry>
     <material name="silver"/>
@@ -20,5 +20,5 @@
     <origin xyz="0 0 0" rpy="0 0 0"/>
     <geometry>
-      <mesh filename="package://linef/models/robot/base_link.stl" scale="0.001 0.001 0.001"/>
+      <mesh filename="package://line_follower_omnidrive/models/robot/base_link.stl" scale="0.001 0.001 0.001"/>
     </geometry>
   </collision>
@@ -33,5 +33,5 @@
     <origin xyz="-0.187451 0.187549 -0.074" rpy="0 0 0"/>
     <geometry>
-      <mesh filename="package://linef/models/robot/upper_panel_1.stl" scale="0.001 0.001 0.001"/>
+      <mesh filename="package://line_follower_omnidrive/models/robot/upper_panel_1.stl" scale="0.001 0.001 0.001"/>
     </geometry>
     <material name="silver"/>
@@ -40,5 +40,5 @@
     <origin xyz="-0.187451 0.187549 -0.074" rpy="0 0 0"/>
     <geometry>
-      <mesh filename="package://linef/models/robot/upper_panel_1.stl" scale="0.001 0.001 0.001"/>
+      <mesh filename="package://line_follower_omnidrive/models/robot/upper_panel_1.stl" scale="0.001 0.001 0.001"/>
     </geometry>
   </collision>
@@ -53,5 +53,5 @@
     <origin xyz="-0.19 0.0 -0.107" rpy="0 0 0"/>
     <geometry>
-      <mesh filename="package://linef/models/robot/camera_1.stl" scale="0.001 0.001 0.001"/>
+      <mesh filename="package://line_follower_omnidrive/models/robot/camera_1.stl" scale="0.001 0.001 0.001"/>
     </geometry>
     <material name="silver"/>
@@ -60,5 +60,5 @@
     <origin xyz="-0.19 0.0 -0.107" rpy="0 0 0"/>
     <geometry>
-      <mesh filename="package://linef/models/robot/camera_1.stl" scale="0.001 0.001 0.001"/>
+      <mesh filename="package://line_follower_omnidrive/models/robot/camera_1.stl" scale="0.001 0.001 0.001"/>
     </geometry>
   </collision>
@@ -73,5 +73,5 @@
     <origin xyz="-0.001209 -0.056886 -0.018723" rpy="0 0 0"/>
     <geometry>
-      <mesh filename="package://linef/models/robot/tyre_l_1.stl" scale="0.001 0.001 0.001"/>
+      <mesh filename="package://line_follower_omnidrive/models/robot/tyre_l_1.stl" scale="0.001 0.001 0.001"/>
     </geometry>
     <material name="silver"/>
@@ -80,5 +80,5 @@
     <origin xyz="-0.001209 -0.056886 -0.018723" rpy="0 0 0"/>
     <geometry>
-      <mesh filename="package://linef/models/robot/tyre_l_1.stl" scale="0.001 0.001 0.001"/>
+      <mesh filename="package://line_follower_omnidrive/models/robot/tyre_l_1.stl" scale="0.001 0.001 0.001"/>
     </geometry>
   </collision>
@@ -93,5 +93,5 @@
     <origin xyz="-0.000109 0.150886 -0.018723" rpy="0 0 0"/>
     <geometry>
-      <mesh filename="package://linef/models/robot/tyre_r_1.stl" scale="0.001 0.001 0.001"/>
+      <mesh filename="package://line_follower_omnidrive/models/robot/tyre_r_1.stl" scale="0.001 0.001 0.001"/>
     </geometry>
     <material name="silver"/>
@@ -100,5 +100,5 @@
     <origin xyz="-0.000109 0.150886 -0.018723" rpy="0 0 0"/>
     <geometry>
-      <mesh filename="package://linef/models/robot/tyre_r_1.stl" scale="0.001 0.001 0.001"/>
+      <mesh filename="package://line_follower_omnidrive/models/robot/tyre_r_1.stl" scale="0.001 0.001 0.001"/>
     </geometry>
   </collision>
